File: kicad/board/board.kicad_pcb (KiCad board)
At the start: 2 copper layers, 126.9 x 103.7 mm, 39 parts

Commit message: updated pcb
Parts:
- D1, D10, D11, D12, D13, D14, D15, D16, D17, D18, D2, D3, D4, D5, D6, D7, D8, D9: value (none) -> 1N914; footprint ComboDiode -> clacken:reversable_diode
- JST1, JST2: value (none) -> Conn_01x02; footprint JST_PH_S2B-PH-K_02x2.00mm_Angled -> clacken:JST_angled
- S1, S10, S11, S12, S13, S14, S15, S16, S17, S18, S2, S3, S4, S5, S6, S7, S8, S9: value (none) -> SW_Push_45deg; footprint PG1350 -> clacken:choc_switches
- gave numbers to parts that had none: 1
Connections:
- D1 pad 1: (no net) -> Row3
- D1 pad 2: (no net) -> Net-(D1-A)
- D10 pad 1: (no net) -> Row3
- D10 pad 2: (no net) -> Net-(D10-A)
- D11 pad 1: (no net) -> Row2
- D11 pad 2: (no net) -> Net-(D11-A)
- D12 pad 1: (no net) -> Row1
- D12 pad 2: (no net) -> Net-(D12-A)
- D13 pad 1: (no net) -> Row3
- D13 pad 2: (no net) -> Net-(D13-A)
- D14 pad 1: (no net) -> Row2
- D14 pad 2: (no net) -> Net-(D14-A)
- D15 pad 1: (no net) -> Row1
- D15 pad 2: (no net) -> Net-(D15-A)
- D16 pad 1: (no net) -> Row4
- D16 pad 2: (no net) -> Net-(D16-A)
- D17 pad 1: (no net) -> Row4
- D17 pad 2: (no net) -> Net-(D17-A)
- D18 pad 1: (no net) -> Row4
- D18 pad 2: (no net) -> Net-(D18-A)
- D2 pad 1: (no net) -> Row2
- D2 pad 2: (no net) -> Net-(D2-A)
- D3 pad 1: (no net) -> Row1
- D3 pad 2: (no net) -> Net-(D3-A)
- D4 pad 1: (no net) -> Row3
- D4 pad 2: (no net) -> Net-(D4-A)
- D5 pad 1: (no net) -> Row2
- D5 pad 2: (no net) -> Net-(D5-A)
- D6 pad 1: (no net) -> Row1
- D6 pad 2: (no net) -> Net-(D6-A)
- D7 pad 1: (no net) -> Row3
- D7 pad 2: (no net) -> Net-(D7-A)
- D8 pad 1: (no net) -> Row2
- D8 pad 2: (no net) -> Net-(D8-A)
- D9 pad 1: (no net) -> Row1
- D9 pad 2: (no net) -> Net-(D9-A)
- JST1 pad 1: (no net) -> Net-(JST1-Pin_1)
- JST1 pad 2: (no net) -> Net-(JST1-Pin_2)
- JST2 pad 1: (no net) -> Net-(JST1-Pin_1)
- JST2 pad 2: (no net) -> Net-(JST1-Pin_2)
- S1 pad 1: (no net) -> Col1
- S1 pad 2: (no net) -> Net-(D1-A)
- S10 pad 1: (no net) -> Col4
- S10 pad 2: (no net) -> Net-(D10-A)
- S11 pad 1: (no net) -> Col4
- S11 pad 2: (no net) -> Net-(D11-A)
- S12 pad 1: (no net) -> Col4
- S12 pad 2: (no net) -> Net-(D12-A)
- S13 pad 1: (no net) -> Col5
- S13 pad 2: (no net) -> Net-(D13-A)
- S14 pad 1: (no net) -> Col5
- S14 pad 2: (no net) -> Net-(D14-A)
- S15 pad 1: (no net) -> Col5
- S15 pad 2: (no net) -> Net-(D15-A)
- S16 pad 1: (no net) -> Col3
- S16 pad 2: (no net) -> Net-(D16-A)
- S17 pad 1: (no net) -> Col4
- S17 pad 2: (no net) -> Net-(D17-A)
- S18 pad 1: (no net) -> Col5
- S18 pad 2: (no net) -> Net-(D18-A)
- S2 pad 1: (no net) -> Col1
- S2 pad 2: (no net) -> Net-(D2-A)
- S3 pad 1: (no net) -> Col1
- S3 pad 2: (no net) -> Net-(D3-A)
- S4 pad 1: (no net) -> Col2
- S4 pad 2: (no net) -> Net-(D4-A)
- S5 pad 1: (no net) -> Col2
- S5 pad 2: (no net) -> Net-(D5-A)
- S6 pad 1: (no net) -> Col2
- S6 pad 2: (no net) -> Net-(D6-A)
- S7 pad 1: (no net) -> Col3
- S7 pad 2: (no net) -> Net-(D7-A)
- S8 pad 1: (no net) -> Col3
- S8 pad 2: (no net) -> Net-(D8-A)
- S9 pad 1: (no net) -> Col3
- S9 pad 2: (no net) -> Net-(D9-A)
